File: kicad/foxboard/foxboard.kicad_pcb (KiCad board)
At the start: 2 copper layers, 356.7 x 159.4 mm, 181 parts, among them J2 USB_C_Receptacle_USB2.0, K1 KEYSW, K10 KEYSW, K11 KEYSW, K12 KEYSW, K13 KEYSW, K14 KEYSW, K15 KEYSW, K16 KEYSW, K17 KEYSW, K18 KEYSW, K19 KEYSW, K2 KEYSW, K20 KEYSW, K21 KEYSW, K22 KEYSW, K23 KEYSW, K24 KEYSW, K25 KEYSW, K26 KEYSW, K27 KEYSW, K28 KEYSW, K29 KEYSW, K3 KEYSW, K30 KEYSW, K31 KEYSW, K32 KEYSW, K33 KEYSW, K34 KEYSW, K35 KEYSW, K36 KEYSW, K37 KEYSW, K38 KEYSW, K39 KEYSW, K4 KEYSW, K40 KEYSW, K41 KEYSW, K42 KEYSW, K43 KEYSW, K44 KEYSW, K45 KEYSW, K46 KEYSW, K47 KEYSW, K48 KEYSW, K49 KEYSW, K5 KEYSW, K50 KEYSW, K51 KEYSW, K52 KEYSW, K53 KEYSW, K54 KEYSW, K55 KEYSW, K56 KEYSW, K57 KEYSW, K58 KEYSW, K59 KEYSW, K6 KEYSW, K60 KEYSW, K61 KEYSW, K62 KEYSW, K63 KEYSW, K64 KEYSW, K65 KEYSW, K66 KEYSW, K67 KEYSW, K68 KEYSW, K69 KEYSW, K7 KEYSW, K70 KEYSW, K71 KEYSW, K72 KEYSW, K73 KEYSW, K74 KEYSW, K75 KEYSW, K76 KEYSW, K77 KEYSW, K78 KEYSW, K79 KEYSW, K8 KEYSW, K80 KEYSW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

Commit message: move teensy and stuff
Parts:
- moved U2 281.7 mm to (301.0, 320.0)
- moved J2 176.8 mm to (12.6, 245.6)
- moved K1 17.0 mm to (5.08, 337.8)
Changed lines of the file:
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@@
   )
   (footprint "teensy:Teensy41" (layer "F.Cu")
-    (at 50.4575 191.185)
+    (at 300.99 320.04)
     (property "Sheetfile" "foxboard.kicad_sch")
     (property "Sheetname" "")
@@
   )
   (footprint "Connector_USB:USB_C_Receptacle_Amphenol_12401548E4-2A" (layer "F.Cu")
-    (at 185.3775 208.475)
+    (at 12.56 245.58)
     (descr "USB TYPE C, RA RCPT PCB, Hybrid, https://www.amphenolcanada.com/StockAvailabilityPrice.aspx?From=&PartNum=12401548E4%7e2A")
     (tags "USB C Type-C Receptacle Hybrid")
@@
   )
   (footprint "PCM_marbastlib-mx:SW_MX_1.25u" (layer "F.Cu")
-    (at -2.54 353.06)
+    (at 5.08 337.82)
     (descr "Footprint for Cherry MX style switches")
     (property "Sheetfile" "foxboard.kicad_sch")

Commit message: update
Parts:
- D2: value D -> D2
- D3: value D -> D3
- moved K9 446.0 mm to (284.5, 355.6)
- moved K10 441.3 mm to (303.5, 355.6)
- moved K11 438.3 mm to (322.6, 355.6)
- moved K38 367.4 mm to (-3.81, 298.4)
- moved K24 367.2 mm to (302.3, 336.6)
- moved K19 360.9 mm to (151.1, 336.6)
- moved K2 350.2 mm to (19.1, 355.6)
- moved K20 347.8 mm to (170.2, 336.6)
- moved K52 337.7 mm to (285.8, 298.4)
- moved K70 337.2 mm to (323.2, 279.4)
- moved K21 336.5 mm to (189.2, 336.6)
- moved K50 331.7 mm to (232.4, 298.4)
- moved K53 331.6 mm to (304.8, 298.4)
- moved K30 328.7 mm to (102.9, 317.5)
- moved K54 327.7 mm to (323.9, 298.4)
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
Commit message: add keyswitch and change some footprints
Parts:
- K1, K2, K3, K5, K6, K7, K8: footprint PCM_marbastlib-mx:SW_MX_1.25u -> PCM_marbastlib-mx:STAB_MX_P_2u
- K25: footprint PCM_marbastlib-mx:STAB_MX_2.25u -> PCM_marbastlib-mx:SW_MX_1.5u
- K37: footprint PCM_marbastlib-xp-plate-mx:Plate_MX_ANSI-ISO-ENTER -> PCM_marbastlib-mx:STAB_MX_2u
- K38, K51: footprint PCM_marbastlib-mx:SW_MX_1.75u -> PCM_marbastlib-mx:SW_MX_1.5u
- K69: footprint PCM_marbastlib-mx:STAB_MX_2.75u -> PCM_marbastlib-mx:STAB_MX_P_2u
- moved K37 14.4 mm to (247.2, 317.5)
- moved K25 4.33 mm to (0.00, 317.5)
- moved K51 2.54 mm to (256.5, 298.4)
- moved K38 1.27 mm to (-2.54, 298.4)
- moved K69 1.27 mm to (252.3, 278.8)

Commit message: update layout
Parts:
- added D87: D, Diode_SMD:D_0201_0603Metric_Pad0.64x0.40mm_HandSolder, F.Cu at (276.4, 289.6)
- added K87: KEYSW, PCM_marbastlib-mx:SW_MX_1u, F.Cu at (284.9, 279.4)
- D2: value D2 -> D
- D3: value D3 -> D
- K1, K2, K3, K5, K6, K7, K8: footprint PCM_marbastlib-mx:STAB_MX_P_2u -> PCM_marbastlib-mx:SW_MX_1.25u
- K12: footprint PCM_marbastlib-xp-plate-mx:Plate_MX_SPLIT-RSHIFT -> PCM_marbastlib-mx:STAB_MX_2.25u
- K25: footprint PCM_marbastlib-mx:SW_MX_1.5u -> PCM_marbastlib-mx:SW_MX_HS_1.5u
- K51: footprint PCM_marbastlib-mx:SW_MX_1.5u -> PCM_marbastlib-mx:SW_MX_1.75u
- K69: footprint PCM_marbastlib-mx:STAB_MX_P_2u -> PCM_marbastlib-mx:STAB_MX_2.75u
- moved K12 3.02 mm to (4.29, 336.6)
- moved K25 2.80 mm to (2.80, 317.5)
- moved K38 1.27 mm to (-2.54, 299.7)
- moved K37 0.79 mm to (246.4, 317.5)
Connections:
- K68 pad 1: Net-(K51-Pad1) -> Net-(K68-Pad1)
- K83 pad 1: unconnected-(K83-Pad1) -> Net-(K68-Pad1)

Commit message: update some footprints and move most diodes into place
Parts:
- moved D25 211.0 mm to (15.0, 309.2)
- moved D38 205.6 mm to (10.1, 289.7)
- moved D55 203.2 mm to (2.54, 271.3)
- moved D56 195.4 mm to (21.6, 271.4)
- moved D26 194.4 mm to (34.5, 309.2)
- moved D39 186.8 mm to (30.8, 289.7)
- moved D27 178.0 mm to (54.4, 309.2)
- moved D57 178.0 mm to (40.5, 271.5)
- moved D40 170.9 mm to (48.5, 289.8)
- moved D54 165.4 mm to (331.3, 290.5)
- moved D28 163.3 mm to (73.0, 309.2)
- moved D58 160.5 mm to (59.8, 271.6)
- moved D41 153.3 mm to (69.1, 289.8)
- moved D53 150.8 mm to (312.0, 290.8)
- moved D29 149.4 mm to (91.9, 309.2)
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Connections:
- D36 pad 2: unconnected-(D36-A-Pad2) -> Net-(D36-A)
- K25 pad 1: (no net) -> Net-(K1-Pad1)
- K25 pad 2: (no net) -> Net-(D25-A)
- K36 pad 2: unconnected-(K36-Pad2) -> Net-(D36-A)

Commit message: update footprints
Parts:
- K51: footprint PCM_marbastlib-mx:SW_MX_1.75u -> PCM_marbastlib-mx:SW_MX_1.25u
- K69: footprint PCM_marbastlib-mx:STAB_MX_2.75u -> PCM_marbastlib-mx:STAB_MX_2u
- moved D51 7.00 mm to (263.7, 290.2)
- moved K51 2.54 mm to (254.0, 298.4)
- moved K69 1.64 mm to (252.3, 278.9)
Changed lines of the file:
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@@
     )
   )
-  (footprint "PCM_marbastlib-mx:STAB_MX_2.75u" (layer "F.Cu")
-    (at 253.89205 278.9174)
-    (descr "Footprint for Cherry Clip/Screw in type stabilizers, 2.75u")
+  (footprint "PCM_marbastlib-mx:STAB_MX_2u" (layer "F.Cu")
+    (at 252.25375 278.9174)
+    (descr "Footprint for Cherry Clip/Screw in type stabilizers, 2u")
     (property "Sheetfile" "foxboard.kicad_sch")
     (property "Sheetname" "")
-    (attr through_hole exclude_from_pos_files)
+    (attr through_hole exclude_from_pos_files exclude_from_bom)
     (fp_text reference "K69" (at 0 0) (layer "F.SilkS") hide
         (effects (font (size 1 1) (thickness 0.15)))
@@
         (effects (font (size 1 1) (thickness 0.15)))
     )
-    (fp_line (start -26.19375 -9.525) (end -26.19375 9.525)
+    (fp_line (start -19.05 -9.525) (end -19.05 9.525)
       (stroke (width 0.12) (type solid)) (layer "Dwgs.User"))
-    (fp_line (start -26.19375 -9.525) (end 26.19375 -9.525)
+    (fp_line (start -19.05 -9.525) (end 19.05 -9.525)
       (stroke (width 0.12) (type solid)) (layer "Dwgs.User"))
-    (fp_line (start -26.19375 9.525) (end 26.19375 9.525)
+    (fp_line (start -19.05 9.525) (end 19.05 9.525)
       (stroke (width 0.12) (type solid)) (layer "Dwgs.User"))
     (fp_line (start -7 -7) (end -5 -7)
@@
     (fp_line (start 7 7) (end 7 5)
       (stroke (width 0.12) (type solid)) (layer "Dwgs.User"))
-    (fp_line (start 26.19375 -9.525) (end 26.19375 9.525)
+    (fp_line (start 19.05 -9.525) (end 19.05 9.525)
       (stroke (width 0.12) (type solid)) (layer "Dwgs.User"))
     (fp_line (start -15.28125 -5.499999) (end -15.28125 7.500001)
@@
     (pad "" np_thru_hole circle (at 11.90625 -6.985) (size 3.048 3.048) (drill 3.048) (layers "*.Cu" "*.Mask"))
     (pad "" np_thru_hole circle (at 11.90625 8.255) (size 3.9878 3.9878) (drill 3.9878) (layers "*.Cu" "*.Mask"))
-    (group "" (id bf4da1a9-9377-4e7c-8cb9-8dd7f6f99009)
+    (group "" (id 9b0b3f10-4e81-4182-afee-985c343a3dae)
       (members
-        1623d7b8-8366-4a36-91ab-963b78cfbb65
-        28f623e2-bb0d-49e9-9adf-ddb3bf288ce9
-        4f929642-a32c-4542-8a39-8201b10e850e
-        7c32e7f6-fe8a-407f-b4f9-8121458f54b3
-        86d5fba0-6175-4528-8282-df6072988444
-        96c4ab4f-df0e-4ef3-b218-b36cc47f6361
-        99463d64-0a04-44c6-9143-0dbf6ee2cca3
-        af428c73-a07b-42d0-a0f4-bf3daf3883ce
+        1263d417-8529-4662-96b0-e53af030510e
+        2173937a-f2c5-4433-a336-fe0027aa2eca
+        44082e26-26d2-4055-8b1e-2dad7523f5ae
+        55efa6b9-3354-47d1-898f-6f0aedea8a93
+        cb91ace8-8eba-4e95-bc6e-7409f041307e
+        d1314675-f56a-46af-9e90-810da2d8afa0
+        d1bf35d7-7846-46e9-b35e-7f41f215a210
+        da951140-9773-42f0-be06-d2e272270397
       )
     )
-    (group "" (id eca2ad65-2a0f-4acd-a530-22d0d0719cbb)
+    (group "" (id da95826a-73ec-4cfb-ab4d-72ad60065779)
       (members
-        3a8481ea-1b75-486f-bcc1-3eeb3732ef13
-        9a05aadb-af9c-4501-b6fb-29f96e32602c
-        a5ab7380-215b-4108-9286-4144b75b584c
-        c3827e8b-01cc-450c-8bcf-43d6533e6635
-        c80dceb0-f19d-4493-99a7-cec64ffa2525
-        d87d52a9-fc25-4a32-99c8-0e03dd64bc1c
-        ea95a392-72a4-4d26-9985-7dbc3cef59c6
-        ed4992dd-2456-4464-93d7-d5bf0444d4b6
+        103d592b-1127-4a42-8deb-e1081741acb2
+        37c24acc-0b3a-45f5-9f0f-57951c9a3fdd
+        4c9f75a9-7605-4c3d-9103-6f4cf2529605
+        8a897439-89fa-422f-bbad-1d8e741f3f05
+        8d189558-fbc7-4ed7-9f25-bf35e2318a36
+        b0fd221e-ff08-42fa-a0d0-12022f162556
+        e2ba7159-f298-45de-9535-f9c6f0cf5ebf
+        e7a0b18c-85fa-452e-923f-e77f7819c4fd
       )
     )
@@
   )
   (footprint "Diode_SMD:D_0201_0603Metric_Pad0.64x0.40mm_HandSolder" (layer "F.Cu")
-    (at 270.7266 290.2204)
+    (at 263.7275 290.2204)
     (descr "Diode SMD 0201 (0603 Metric), square (rectangular) end terminal, IPC_7351 nominal, (Body size source: https://www.vishay.com/docs/20052/crcw0201e3.pdf), generated with kicad-footprint-generator")
     (tags "diode handsolder")
@@
     )
   )
-  (footprint "PCM_marbastlib-mx:SW_MX_1.75u" (layer "F.Cu")
-    (at 256.54 298.45)
+  (footprint "PCM_marbastlib-mx:SW_MX_1.25u" (layer "F.Cu")
+    (at 254 298.45)
     (descr "Footprint for Cherry MX style switches")
     (property "Sheetfile" "foxboard.kicad_sch")
     (property "Sheetname" "")
-    (attr through_hole exclude_from_pos_files)
+    (attr through_hole exclude_from_pos_files exclude_from_bom)
     (fp_text reference "K51" (at 0 3.175) (layer "Dwgs.User") hide
         (effects (font (size 1 1) (thickness 0.15)))
@@
         (effects (font (size 1 1) (thickness 0.15)))
     )
-    (fp_line (start -16.66875 -9.525) (end -16.66875 9.525)
+    (fp_line (start -11.90625 -9.525) (end -11.90625 9.525)
       (stroke (width 0.12) (type solid)) (layer "Dwgs.User"))
-    (fp_line (start -16.66875 9.525) (end 16.66875 9.525)
+    (fp_line (start -11.90625 9.525) (end 11.90625 9.525)
       (stroke (width 0.12) (type solid)) (layer "Dwgs.User"))
-    (fp_line (start 16.66875 -9.525) (end -16.66875 -9.525)
+    (fp_line (start 11.90625 -9.525) (end -11.90625 -9.525)
       (stroke (width 0.12) (type solid)) (layer "Dwgs.User"))
-    (fp_line (start 16.66875 9.525) (end 16.66875 -9.525)
+    (fp_line (start 11.90625 9.525) (end 11.90625 -9.525)
       (stroke (width 0.12) (type solid)) (layer "Dwgs.User"))
     (fp_line (start -7 6.5) (end -7 -6.5)

Commit message: finish layout
Parts:
- moved D71 205.2 mm to (1.02, 243.3)
- moved C3 187.0 mm to (16.0, 264.2), turned to 90 degrees
- moved C4 184.8 mm to (17.7, 264.2), turned to 90 degrees
- moved C5 182.6 mm to (19.5, 264.2), turned to 90 degrees
- moved C6 180.4 mm to (21.2, 264.2), turned to 90 degrees
- moved C7 178.2 mm to (23.0, 264.2), turned to 90 degrees
- moved R5 174.9 mm to (11.9, 257.6)
- moved R6 174.9 mm to (11.9, 260.5)
- moved D72 168.3 mm to (38.9, 243.5)
- moved D70 154.6 mm to (330.0, 271.5)
- moved D73 149.8 mm to (57.9, 243.5)
- moved D69 140.5 mm to (311.7, 271.6)
- moved D86 133.0 mm to (327.2, 243.7)
- moved D74 130.7 mm to (77.6, 243.5)
- moved D85 118.4 mm to (310.8, 243.6)
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
Commit message: update footprints
Parts:
- K25: footprint PCM_marbastlib-mx:SW_MX_HS_1.5u -> PCM_marbastlib-mx:SW_MX_HS_1.75u
- moved K25 2.80 mm to (0.00, 317.5)
Changed lines of the file:
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@@
       (net 69 "Net-(D62-A)") (pintype "passive"))
   )
-  (footprint "PCM_marbastlib-mx:SW_MX_HS_1.5u" (layer "F.Cu")
-    (at 2.8 317.5)
+  (footprint "PCM_marbastlib-mx:SW_MX_HS_1.75u" (layer "F.Cu")
+    (at 0 317.5)
     (descr "Footprint for Cherry MX style switches with Kailh hotswap socket")
     (property "Sheetfile" "foxboard.kicad_sch")
@@
     (fp_arc (start 4.085176 -6.75022) (mid 5.49939 -6.164434) (end 6.085176 -4.75022)
       (stroke (width 0.15) (type solid)) (layer "F.SilkS"))
-    (fp_line (start -14.2875 -9.525) (end 14.2875 -9.525)
+    (fp_line (start -16.66875 -9.525) (end 16.66875 -9.525)
       (stroke (width 0.12) (type solid)) (layer "Dwgs.User"))
-    (fp_line (start -14.2875 9.525) (end -14.2875 -9.525)
+    (fp_line (start -16.66875 9.525) (end -16.66875 -9.525)
       (stroke (width 0.12) (type solid)) (layer "Dwgs.User"))
-    (fp_line (start 14.2875 -9.525) (end 14.2875 9.525)
+    (fp_line (start 16.66875 -9.525) (end 16.66875 9.525)
       (stroke (width 0.12) (type solid)) (layer "Dwgs.User"))
-    (fp_line (start 14.2875 9.525) (end -14.2875 9.525)
+    (fp_line (start 16.66875 9.525) (end -16.66875 9.525)
       (stroke (width 0.12) (type solid)) (layer "Dwgs.User"))
     (fp_line (start -7 -6.5) (end -7 6.5)
