File: kicad/foxboard/foxboard.kicad_pcb (KiCad board)
At the start: 2 copper layers, 40.2 x 15 mm, 184 parts, among them J2 USB_C_Receptacle_USB2.0, K1 KEYSW, K10 KEYSW, K11 KEYSW, K12 KEYSW, K13 KEYSW, K14 KEYSW, K15 KEYSW, K16 KEYSW, K17 KEYSW, K18 KEYSW, K19 KEYSW, K2 KEYSW, K20 KEYSW, K21 KEYSW, K22 KEYSW, K23 KEYSW, K24 KEYSW, K25 KEYSW, K26 KEYSW, K27 KEYSW, K28 KEYSW, K29 KEYSW, K3 KEYSW, K30 KEYSW, K31 KEYSW, K32 KEYSW, K33 KEYSW, K34 KEYSW, K35 KEYSW, K36 KEYSW, K37 KEYSW, K38 KEYSW, K39 KEYSW, K4 KEYSW, K40 KEYSW, K41 KEYSW, K42 KEYSW, K43 KEYSW, K44 KEYSW, K45 KEYSW, K46 KEYSW, K47 KEYSW, K48 KEYSW, K49 KEYSW, K5 KEYSW, K50 KEYSW, K51 KEYSW, K52 KEYSW, K53 KEYSW, K54 KEYSW, K55 KEYSW, K56 KEYSW, K57 KEYSW, K58 KEYSW, K59 KEYSW, K6 KEYSW, K60 KEYSW, K61 KEYSW, K62 KEYSW, K63 KEYSW, K64 KEYSW, K65 KEYSW, K66 KEYSW, K67 KEYSW, K68 KEYSW, K69 KEYSW, K7 KEYSW, K70 KEYSW, K71 KEYSW, K72 KEYSW, K73 KEYSW, K74 KEYSW, K75 KEYSW, K76 KEYSW, K77 KEYSW, K78 KEYSW, K79 KEYSW, K8 KEYSW, K80 KEYSW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

Commit message: add rows
Parts:
- removed the D37 at (256.4, 297.9)
- added D37: D, Diode_SMD:D_0201_0603Metric_Pad0.64x0.40mm_HandSolder, F.Cu at (1.14, 0.38)
- added D37: D, Diode_SMD:D_0201_0603Metric_Pad0.64x0.40mm_HandSolder, B.Cu at (257.0, 297.2)
- moved D68 53.7 mm to (296.7, 259.5)
- moved D69 47.5 mm to (246.8, 259.6)
- moved D51 2.72 mm to (258.7, 279.4)
- moved D54 1.21 mm to (315.4, 279.4)
Connections:
- D38 pad 1: Net-(D37-K) -> Net-(D38-K)
- D39 pad 1: Net-(D37-K) -> Net-(D38-K)
- D40 pad 1: Net-(D37-K) -> Net-(D38-K)
- D41 pad 1: Net-(D37-K) -> Net-(D38-K)
- D42 pad 1: Net-(D37-K) -> Net-(D38-K)
- D43 pad 1: Net-(D37-K) -> Net-(D38-K)
- D44 pad 1: Net-(D37-K) -> Net-(D38-K)
- D45 pad 1: Net-(D37-K) -> Net-(D38-K)
- D46 pad 1: Net-(D37-K) -> Net-(D38-K)
- D47 pad 1: Net-(D37-K) -> Net-(D38-K)
- D48 pad 1: Net-(D37-K) -> Net-(D38-K)
- D49 pad 1: Net-(D37-K) -> Net-(D38-K)
- D50 pad 1: Net-(D37-K) -> Net-(D38-K)
- D51 pad 1: Net-(D37-K) -> Net-(D38-K)
- D52 pad 1: Net-(D37-K) -> Net-(D38-K)
- D53 pad 1: Net-(D37-K) -> Net-(D38-K)
- D54 pad 1: Net-(D54-K) -> Net-(D38-K)
- D55 pad 1: Net-(D54-K) -> Net-(D55-K)
- D56 pad 1: Net-(D54-K) -> Net-(D55-K)
- D57 pad 1: Net-(D54-K) -> Net-(D55-K)
- D58 pad 1: Net-(D54-K) -> Net-(D55-K)
- D59 pad 1: Net-(D54-K) -> Net-(D55-K)
- D60 pad 1: Net-(D54-K) -> Net-(D55-K)
- D61 pad 1: Net-(D54-K) -> Net-(D55-K)
- D62 pad 1: Net-(D54-K) -> Net-(D55-K)
- D63 pad 1: Net-(D54-K) -> Net-(D55-K)
- D64 pad 1: Net-(D54-K) -> Net-(D55-K)
- D65 pad 1: Net-(D54-K) -> Net-(D55-K)
- D66 pad 1: Net-(D54-K) -> Net-(D55-K)
- D67 pad 1: Net-(D54-K) -> Net-(D55-K)
- D68 pad 1: Net-(D54-K) -> Net-(D55-K)
- D69 pad 1: Net-(D54-K) -> Net-(D55-K)
- D70 pad 1: Net-(D54-K) -> Net-(D55-K)
- D70 pad 2: unconnected-(D70-A-Pad2) -> Net-(D70-A)
- D87 pad 1: Net-(D54-K) -> Net-(D55-K)
- K1 pad 1: Net-(U2-39_MISO1_OUT1A) -> Net-(K1-Pad1)
- K10 pad 1: Net-(U2-1_TX1_CTX2_MISO1) -> Net-(K10-Pad1)
- K11 pad 1: Net-(U2-0_RX1_CRX2_CS1) -> Net-(K11-Pad1)
- K13 pad 1: Net-(U2-40_A16) -> Net-(K13-Pad1)
- K14 pad 1: Net-(U2-41_A17) -> Net-(K14-Pad1)
- K15 pad 1: Net-(U2-13_SCK_LED) -> Net-(K15-Pad1)
- K16 pad 1: Net-(U2-14_A0_TX3_SPDIF_OUT) -> Net-(K16-Pad1)
- K17 pad 1: Net-(U2-15_A1_RX3_SPDIF_IN) -> Net-(K17-Pad1)
- K18 pad 1: Net-(U2-16_A2_RX4_SCL1) -> Net-(K18-Pad1)
- K19 pad 1: Net-(U2-17_A3_TX4_SDA1) -> Net-(K19-Pad1)
- K2 pad 1: Net-(U2-40_A16) -> Net-(K13-Pad1)
- K20 pad 1: Net-(U2-8_TX2_IN1) -> Net-(K20-Pad1)
- K21 pad 1: Net-(U2-7_RX2_OUT1A) -> Net-(K21-Pad1)
- K22 pad 1: Net-(U2-6_OUT1D) -> Net-(K22-Pad1)
- K24 pad 1: Net-(U2-1_TX1_CTX2_MISO1) -> Net-(K10-Pad1)
- K26 pad 1: Net-(U2-40_A16) -> Net-(K13-Pad1)
- K27 pad 1: Net-(U2-41_A17) -> Net-(K14-Pad1)
- K28 pad 1: Net-(U2-13_SCK_LED) -> Net-(K15-Pad1)
- K29 pad 1: Net-(U2-14_A0_TX3_SPDIF_OUT) -> Net-(K16-Pad1)
- K3 pad 1: Net-(U2-41_A17) -> Net-(K14-Pad1)
- K30 pad 1: Net-(U2-15_A1_RX3_SPDIF_IN) -> Net-(K17-Pad1)
- K31 pad 1: Net-(U2-16_A2_RX4_SCL1) -> Net-(K18-Pad1)
- K32 pad 1: Net-(U2-17_A3_TX4_SDA1) -> Net-(K19-Pad1)
- K33 pad 1: Net-(U2-8_TX2_IN1) -> Net-(K20-Pad1)
- K34 pad 1: Net-(U2-7_RX2_OUT1A) -> Net-(K21-Pad1)
- K35 pad 1: Net-(U2-6_OUT1D) -> Net-(K22-Pad1)
- K38 pad 1: Net-(U2-40_A16) -> Net-(K13-Pad1)
- K39 pad 1: Net-(U2-41_A17) -> Net-(K14-Pad1)
- K4 pad 1: Net-(U2-15_A1_RX3_SPDIF_IN) -> Net-(K17-Pad1)
- K40 pad 1: Net-(U2-13_SCK_LED) -> Net-(K15-Pad1)
- K41 pad 1: Net-(U2-14_A0_TX3_SPDIF_OUT) -> Net-(K16-Pad1)
- K42 pad 1: Net-(U2-15_A1_RX3_SPDIF_IN) -> Net-(K17-Pad1)
- K43 pad 1: Net-(U2-16_A2_RX4_SCL1) -> Net-(K18-Pad1)
- K44 pad 1: Net-(U2-17_A3_TX4_SDA1) -> Net-(K19-Pad1)
- K45 pad 1: Net-(U2-8_TX2_IN1) -> Net-(K20-Pad1)
- K45 pad 2: Net-(D46-A) -> Net-(D45-A)
- K46 pad 1: Net-(U2-7_RX2_OUT1A) -> Net-(K21-Pad1)
- K46 pad 2: Net-(D47-A) -> Net-(D46-A)
- K47 pad 2: Net-(D48-A) -> Net-(D47-A)
- K48 pad 1: Net-(U2-6_OUT1D) -> Net-(K22-Pad1)
- K48 pad 2: Net-(D49-A) -> Net-(D48-A)
- K49 pad 2: Net-(D50-A) -> Net-(D49-A)
- K5 pad 1: Net-(U2-8_TX2_IN1) -> Net-(K20-Pad1)
- K50 pad 2: Net-(D45-A) -> Net-(D50-A)
- K51 pad 1: Net-(U2-2_OUT2) -> Net-(K51-Pad1)
- K52 pad 1: Net-(U2-1_TX1_CTX2_MISO1) -> Net-(K52-Pad1)
- K53 pad 1: Net-(U2-0_RX1_CRX2_CS1) -> Net-(K10-Pad1)
- K54 pad 1: Net-(U2-39_MISO1_OUT1A) -> Net-(K1-Pad1)
- K55 pad 1: Net-(U2-40_A16) -> Net-(K13-Pad1)
- K56 pad 1: Net-(U2-41_A17) -> Net-(K14-Pad1)
- K57 pad 1: Net-(U2-13_SCK_LED) -> Net-(K15-Pad1)
- K58 pad 1: Net-(U2-14_A0_TX3_SPDIF_OUT) -> Net-(K16-Pad1)
- K59 pad 1: Net-(U2-15_A1_RX3_SPDIF_IN) -> Net-(K17-Pad1)
- K6 pad 1: Net-(U2-7_RX2_OUT1A) -> Net-(K21-Pad1)
- K60 pad 1: Net-(U2-16_A2_RX4_SCL1) -> Net-(K18-Pad1)
- K61 pad 1: Net-(U2-17_A3_TX4_SDA1) -> Net-(K19-Pad1)
- K62 pad 1: Net-(U2-8_TX2_IN1) -> Net-(K20-Pad1)
- K63 pad 1: Net-(U2-7_RX2_OUT1A) -> Net-(K21-Pad1)
- K65 pad 1: Net-(U2-6_OUT1D) -> Net-(K22-Pad1)
- K68 pad 1: Net-(U2-3_LRCLK2) -> Net-(K51-Pad1)
- K7 pad 1: Net-(U2-6_OUT1D) -> Net-(K22-Pad1)
- K70 pad 1: Net-(U2-0_RX1_CRX2_CS1) -> Net-(K11-Pad1)
- K70 pad 2: unconnected-(K70-Pad2) -> Net-(D70-A)
- K71 pad 1: Net-(U2-39_MISO1_OUT1A) -> Net-(K1-Pad1)
- K72 pad 1: Net-(U2-40_A16) -> Net-(K13-Pad1)
- K73 pad 1: Net-(U2-41_A17) -> Net-(K14-Pad1)
- K74 pad 1: Net-(U2-14_A0_TX3_SPDIF_OUT) -> Net-(K16-Pad1)
- K75 pad 1: Net-(U2-15_A1_RX3_SPDIF_IN) -> Net-(K17-Pad1)
- K76 pad 1: Net-(U2-16_A2_RX4_SCL1) -> Net-(K18-Pad1)
- K77 pad 1: Net-(U2-17_A3_TX4_SDA1) -> Net-(K19-Pad1)
- K78 pad 1: Net-(U2-8_TX2_IN1) -> Net-(K20-Pad1)
- K79 pad 1: Net-(U2-7_RX2_OUT1A) -> Net-(K21-Pad1)
- K80 pad 1: Net-(U2-6_OUT1D) -> Net-(K22-Pad1)
- K81 pad 1: Net-(U2-5_IN2) -> unconnected-(K81-Pad1)
- K82 pad 1: Net-(U2-4_BCLK2) -> unconnected-(K82-Pad1)
- K83 pad 1: Net-(U2-3_LRCLK2) -> Net-(K51-Pad1)
- K84 pad 1: Net-(U2-2_OUT2) -> Net-(K52-Pad1)
- K85 pad 1: Net-(U2-1_TX1_CTX2_MISO1) -> Net-(K10-Pad1)
- K86 pad 1: Net-(U2-0_RX1_CRX2_CS1) -> Net-(K11-Pad1)
- K87 pad 1: Net-(U2-2_OUT2) -> Net-(K52-Pad1)
- K9 pad 1: Net-(U2-2_OUT2) -> Net-(K52-Pad1)
- U2 pad 10: Net-(U2-8_TX2_IN1) -> unconnected-(U2-8_TX2_IN1-Pad10)
- U2 pad 17: unconnected-(U2-25_A11_RX6_SDA2-Pad17) -> Net-(D25-K)
- U2 pad 2: Net-(U2-0_RX1_CRX2_CS1) -> unconnected-(U2-0_RX1_CRX2_CS1-Pad2)
- U2 pad 22: unconnected-(U2-30_CRX3-Pad22) -> Net-(D38-K)
- U2 pad 23: unconnected-(U2-31_CTX3-Pad23) -> Net-(D12-K)
- U2 pad 24: unconnected-(U2-32_OUT1B-Pad24) -> Net-(D1-K)
- U2 pad 25: Net-(D1-K) -> Net-(D71-K)
- U2 pad 26: Net-(D12-K) -> Net-(D55-K)
- U2 pad 27: Net-(D25-K) -> unconnected-(U2-35_TX8-Pad27)
- U2 pad 28: Net-(D37-K) -> unconnected-(U2-36_CS-Pad28)
- U2 pad 29: Net-(D54-K) -> unconnected-(U2-37_CS-Pad29)
- U2 pad 3: Net-(U2-1_TX1_CTX2_MISO1) -> unconnected-(U2-1_TX1_CTX2_MISO1-Pad3)
- U2 pad 30: Net-(D71-K) -> unconnected-(U2-38_CS1_IN1-Pad30)
- U2 pad 31: Net-(U2-39_MISO1_OUT1A) -> unconnected-(U2-39_MISO1_OUT1A-Pad31)
- U2 pad 32: Net-(U2-40_A16) -> unconnected-(U2-40_A16-Pad32)
- U2 pad 33: Net-(U2-41_A17) -> unconnected-(U2-41_A17-Pad33)
- U2 pad 35: Net-(U2-13_SCK_LED) -> unconnected-(U2-13_SCK_LED-Pad35)
- U2 pad 36: Net-(U2-14_A0_TX3_SPDIF_OUT) -> unconnected-(U2-14_A0_TX3_SPDIF_OUT-Pad36)
- U2 pad 37: Net-(U2-15_A1_RX3_SPDIF_IN) -> unconnected-(U2-15_A1_RX3_SPDIF_IN-Pad37)
- U2 pad 38: Net-(U2-16_A2_RX4_SCL1) -> unconnected-(U2-16_A2_RX4_SCL1-Pad38)
- U2 pad 39: Net-(U2-17_A3_TX4_SDA1) -> unconnected-(U2-17_A3_TX4_SDA1-Pad39)
- U2 pad 4: Net-(U2-2_OUT2) -> unconnected-(U2-2_OUT2-Pad4)
- U2 pad 5: Net-(U2-3_LRCLK2) -> unconnected-(U2-3_LRCLK2-Pad5)
- U2 pad 6: Net-(U2-4_BCLK2) -> unconnected-(U2-4_BCLK2-Pad6)
- U2 pad 7: Net-(U2-5_IN2) -> unconnected-(U2-5_IN2-Pad7)
- U2 pad 8: Net-(U2-6_OUT1D) -> unconnected-(U2-6_OUT1D-Pad8)
- U2 pad 9: Net-(U2-7_RX2_OUT1A) -> unconnected-(U2-7_RX2_OUT1A-Pad9)
Routing:
- net Net-(D71-K): track 0.00 -> 450.5 mm
- net Net-(D55-K): track 0.00 -> 378.8 mm
- net Net-(D38-K): track 0.00 -> 366.7 mm
- net Net-(D1-K): track 0.00 -> 356.0 mm
- net Net-(D12-K): track 0.00 -> 314.5 mm
- net Net-(D25-K): track 0.00 -> 311.4 mm
- net Net-(D38-A): track 0.00 -> 10.1 mm
- net Net-(D87-A): track 0.00 -> 8.58 mm
- net Net-(D51-A): track 0.00 -> 8.56 mm
- net Net-(D5-A): track 0.00 -> 8.30 mm
- net Net-(D8-A): track 0.00 -> 7.84 mm
- net Net-(D7-A): track 0.00 -> 7.56 mm
- net Net-(D6-A): track 0.00 -> 7.26 mm
- net Net-(D18-A): track 0.00 -> 6.46 mm
- net Net-(D75-A): track 0.00 -> 6.45 mm
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
Commit message: add few rows update eeschema
Parts:
- removed K37: KEYSW, PCM_marbastlib-mx:STAB_MX_ISO
- moved D56 3.08 mm to (13.1, 261.6)
- moved D55 2.21 mm to (-10.6, 259.1)
- moved D39 1.51 mm to (23.3, 279.4)
- moved D38 0.32 mm to (2.97, 279.4)
- moved K12 0.18 mm to (-5.08, 325.1)
Connections:
- K11 pad 1: Net-(K11-Pad1) -> Net-(U2-35_TX8)
- K40 pad 1: Net-(K15-Pad1) -> Net-(K14-Pad1)
- K41 pad 1: Net-(K16-Pad1) -> Net-(K15-Pad1)
- K42 pad 1: Net-(K17-Pad1) -> Net-(K16-Pad1)
- K43 pad 1: Net-(K18-Pad1) -> Net-(K17-Pad1)
- K44 pad 1: Net-(K19-Pad1) -> Net-(K18-Pad1)
- K45 pad 1: Net-(K20-Pad1) -> Net-(K19-Pad1)
- K46 pad 1: Net-(K21-Pad1) -> Net-(K20-Pad1)
- K47 pad 1: unconnected-(K47-Pad1) -> Net-(K21-Pad1)
- K57 pad 1: Net-(K15-Pad1) -> Net-(K14-Pad1)
- K58 pad 1: Net-(K16-Pad1) -> Net-(K15-Pad1)
- K59 pad 1: Net-(K17-Pad1) -> Net-(K16-Pad1)
- K60 pad 1: Net-(K18-Pad1) -> Net-(K17-Pad1)
- K61 pad 1: Net-(K19-Pad1) -> Net-(K18-Pad1)
- K62 pad 1: Net-(K20-Pad1) -> Net-(K19-Pad1)
- K63 pad 1: Net-(K21-Pad1) -> Net-(K20-Pad1)
- K64 pad 1: unconnected-(K64-Pad1) -> Net-(K21-Pad1)
- K70 pad 1: Net-(K11-Pad1) -> Net-(U2-35_TX8)
- K86 pad 1: Net-(K11-Pad1) -> Net-(U2-35_TX8)
- U2 pad 27: unconnected-(U2-35_TX8-Pad27) -> Net-(U2-35_TX8)
Routing:
- net Net-(K22-Pad1): track 0.00 -> 139.9 mm
- net Net-(K21-Pad1): track 0.00 -> 130.3 mm
- net Net-(K20-Pad1): track 0.00 -> 125.6 mm
- net Net-(K17-Pad1): track 0.00 -> 115.6 mm
- net Net-(K18-Pad1): track 0.00 -> 99.7 mm
- net Net-(K19-Pad1): track 0.00 -> 99.7 mm
- net Net-(K16-Pad1): track 0.00 -> 95.7 mm
- net Net-(U2-35_TX8): track 0.00 -> 28.7 mm
- net Net-(D55-K): track 378.8 -> 383.4 mm
- net Net-(D39-A): track 5.24 -> 6.83 mm
- net Net-(D56-A): track 4.77 -> 6.23 mm
- net Net-(D38-K): track 366.7 -> 368.0 mm
- net Net-(D55-A): track 4.61 -> 3.96 mm
