File: kicad/foxboard/foxboard.kicad_sch (KiCad schematic)
At the start: 210 parts, among them J1 Conn_01x02, J3 SWD, J5 USB_C_Receptacle_USB2.0_14P, K1 KEYSW, K10 KEYSW, K11 KEYSW, K12 KEYSW, K13 KEYSW, K14 KEYSW, K15 KEYSW, K16 KEYSW, K17 KEYSW, K18 KEYSW, K19 KEYSW, K2 KEYSW, K20 KEYSW, K21 KEYSW, K22 KEYSW, K23 KEYSW, K24 KEYSW, K25 KEYSW, K26 KEYSW, K27 KEYSW, K28 KEYSW, K29 KEYSW, K3 KEYSW, K30 KEYSW, K31 KEYSW, K32 KEYSW, K33 KEYSW, K34 KEYSW, K35 KEYSW, K36 KEYSW, K37 KEYSW, K38 KEYSW, K39 KEYSW, K4 KEYSW, K40 KEYSW, K41 KEYSW, K42 KEYSW, K43 KEYSW, K44 KEYSW, K45 KEYSW, K46 KEYSW, K47 KEYSW, K48 KEYSW, K49 KEYSW, K5 KEYSW, K50 KEYSW, K51 KEYSW, K52 KEYSW, K53 KEYSW, K54 KEYSW, K55 KEYSW, K56 KEYSW, K57 KEYSW, K58 KEYSW, K59 KEYSW, K6 KEYSW, K60 KEYSW, K61 KEYSW, K62 KEYSW, K63 KEYSW, K64 KEYSW, K65 KEYSW, K66 KEYSW, K67 KEYSW, K68 KEYSW, K69 KEYSW, K7 KEYSW, K70 KEYSW, K71 KEYSW, K72 KEYSW, K73 KEYSW, K74 KEYSW, K75 KEYSW, K76 KEYSW, K77 KEYSW, K78 KEYSW, K79 KEYSW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

Commit message: finish matrix
Parts:
- removed D1, D10, D11, D12, D13, D14, D15, D16, D17, D18, D19, D2, D20, D21, D22, D23, D24, D25, D26, D27, D28, D29, D3, D30, D31, D32, D33, D34, D35, D36, D37, D38, D39, D4, D40, D41, D42, D43, D44, D45, D46, D47, D48, D49, D5, D50, D51, D52, D53, D54, D55, D56, D57, D58, D59, D6, D60, D61, D62, D63, D64, D65, D66, D67, D68, D69, D7, D70, D71, D72, D73, D74, D75, D76, D77, D78, D79, D8, D80, D81, D82, D83, D84, D85, D86, D87, D9: D, 1N4148:DIOAD753W49L380D172B, symbol Device:D
- added D1, D10, D11, D12, D13, D14, D15, D16, D17, D18, D19, D2, D20, D21, D22, D23, D24, D25, D26, D27, D28, D29, D3, D30, D31, D32, D33, D34, D35, D36, D37, D38, D39, D4, D40, D41, D42, D43, D44, D45, D46, D47, D48, D49, D5, D50, D51, D52, D53, D54, D55, D56, D57, D58, D59, D6, D60, D61, D62, D63, D64, D65, D66, D67, D68, D69, D7, D70, D71, D72, D73, D74, D75, D76, D77, D78, D79, D8, D80, D81, D82, D83, D84, D85, D86, D88, D9: 1N914, Diode_THT:D_DO-35_SOD27_P7.62mm_Horizontal, symbol Diode:1N914
Connections:
- net row 1: now also D1.1 (K), D10.1 (K), D11.1 (K), D12.1 (K), D13.1 (K), D14.1 (K), D15.1 (K), D16.1 (K), D2.1 (K), D3.1 (K), D4.1 (K), D5.1 (K), D6.1 (K), D7.1 (K), D8.1 (K), D9.1 (K)
- net row 2: now also D17.1 (K), D18.1 (K), D19.1 (K), D20.1 (K), D21.1 (K), D22.1 (K), D23.1 (K), D24.1 (K), D25.1 (K), D26.1 (K), D27.1 (K), D28.1 (K), D29.1 (K), D30.1 (K), D31.1 (K), D32.1 (K), D33.1 (K)
- net row 3: now also D34.1 (K), D35.1 (K), D36.1 (K), D37.1 (K), D38.1 (K), D39.1 (K), D40.1 (K), D41.1 (K), D42.1 (K), D43.1 (K), D44.1 (K), D46.1 (K), D47.1 (K), D48.1 (K), D49.1 (K), D50.1 (K), D88.1 (K)
- net row 4: now also D45.1 (K), D51.1 (K), D52.1 (K), D53.1 (K), D54.1 (K), D55.1 (K), D56.1 (K), D57.1 (K), D58.1 (K), D59.1 (K), D60.1 (K), D61.1 (K), D62.1 (K)
- net row 5: now also D64.1 (K), D65.1 (K), D66.1 (K), D67.1 (K), D68.1 (K), D69.1 (K), D70.1 (K), D71.1 (K), D72.1 (K), D73.1 (K), D74.1 (K), D75.1 (K), D76.1 (K)
- net row 6: now also D63.1 (K), D77.1 (K), D78.1 (K), D79.1 (K), D80.1 (K), D81.1 (K), D82.1 (K), D83.1 (K), D84.1 (K), D85.1 (K), D86.1 (K)
- net at K12.2: now also D12.2 (A)
- net at K14.2: now also D14.2 (A)
- net at K50.2: now also D88.2 (A)
- net at K83.2: now also D82.2 (A)
- net at K22.2: now also D23.2 (A)
- net at K80.2: now also D79.2 (A)
- net at K31.2: now also D31.2 (A)
- net at K9.2: now also D9.2 (A)
- net at K15.2: now also D15.2 (A)
- net at K30.2: now also D30.2 (A)
- net at K63.2: now also D62.2 (A)
- net at K70.2: now also D70.2 (A)
- net at K76.2: now also D64.2 (A)
- net at K41.2: now also D41.2 (A)
- net at K26.2: now also D26.2 (A)
- net at K27.2: now also D27.2 (A)
- net at K10.2: now also D10.2 (A)
- net at K8.2: now also D8.2 (A)
- net at K73.2: now also D67.2 (A)
- net at K66.2: now also D74.2 (A)
- net at K81.2: now also D80.2 (A)
- net at K21.2: now also D22.2 (A)
- net at K18.2: now also D18.2 (A)
- net at K57.2: now also D56.2 (A)
- net at K2.2: now also D2.2 (A)
- net at K55.2: now also D54.2 (A)
- net at K65.2: now also D75.2 (A)
- net at K44.2: now also D44.2 (A)
- net at K33.2: now also D33.2 (A)
- net at K75.2: now also D65.2 (A)
- net at K45.2: now also D46.2 (A)
- net at K36.2: now also D36.2 (A)
- net at K25.2: now also D25.2 (A)
- net at K86.2: now also D85.2 (A)
- net at K43.2: now also D43.2 (A)
- net at K56.2: now also D55.2 (A)
- net at K64.2: now also D76.2 (A)
- net at K23.2: now also D20.2 (A)
- net at K79.2: now also D78.2 (A)
- net at K34.2: now also D34.2 (A)
- net at K1.2: now also D1.2 (A)
- net at K28.2: now also D28.2 (A)
- net at K68.2: now also D72.2 (A)
- net at K77.2: now also D63.2 (A)
- net at K71.2: now also D69.2 (A)
- net at K51.2: now also D45.2 (A)
- net at K37.2: now also D37.2 (A)
- net at K16.2: now also D16.2 (A)
- net at K78.2: now also D77.2 (A)
- net at K53.2: now also D52.2 (A)
- net at K49.2: now also D50.2 (A)
- net at K47.2: now also D48.2 (A)
- net at K32.2: now also D32.2 (A)
- net at K6.2: now also D6.2 (A)
- net at K46.2: now also D47.2 (A)
- net at K7.2: now also D7.2 (A)
- net at K4.2: now also D4.2 (A)
- net at K35.2: now also D35.2 (A)
- net at K24.2: now also D24.2 (A)
- net at K3.2: now also D3.2 (A)
- net at K58.2: now also D57.2 (A)
- net at K84.2: now also D83.2 (A)
- net at K59.2: now also D58.2 (A)
- net at K52.2: now also D51.2 (A)
- net at K13.2: now also D13.2 (A)
- net at K20.2: now also D21.2 (A)
- net at K11.2: now also D11.2 (A)
- net at K61.2: now also D60.2 (A)
- net at K60.2: now also D59.2 (A)
- net at K42.2: now also D42.2 (A)
- net at K5.2: now also D5.2 (A)
- net at K87.2: now also D86.2 (A)
- net at K69.2: now also D71.2 (A)
- net at K62.2: now also D61.2 (A)
- net at K48.2: now also D49.2 (A)
- net at K29.2: now also D29.2 (A)
- net at K72.2: now also D68.2 (A)
- net at K54.2: now also D53.2 (A)
- net at K82.2: now also D81.2 (A)
- net at K67.2: now also D73.2 (A)
- net at K40.2: now also D40.2 (A)
- net at K19.2: now also D19.2 (A)
- net at K39.2: now also D39.2 (A)
- net at K38.2: now also D38.2 (A)
- net at K17.2: now also D17.2 (A)
- net at K85.2: now also D84.2 (A)
- net at K74.2: now also D66.2 (A)
